File: pcb/pcb.kicad_sch (KiCad schematic)
At the start: 6 parts, among them J1 Connector, USB-TYPE-C-16P, U1 MCP1700x-330xxTT

Commit message: more pcb work
Parts:
- removed U1: MCP1700x-330xxTT, Package_TO_SOT_SMD:SOT-23, symbol Regulator_Linear:MCP1700x-330xxTT
- added C10, C11, C12, C14, C15, C3, C5, C6, C7, C8, C9: 0.1uF, Capacitor_SMD:C_0805_2012Metric, symbol Device:C
- added C13, C4: 1uF, Capacitor_SMD:C_0805_2012Metric, symbol Device:C
- added C16, C17: 15pF, Capacitor_SMD:C_0805_2012Metric, symbol Device:C
- added R3, R4: 27, Resistor_SMD:R_0603_1608Metric, symbol Device:R
- added R5: 10k, Resistor_SMD:R_0603_1608Metric, symbol Device:R
- added R6, R7: 1k, Resistor_SMD:R_0603_1608Metric, symbol Device:R
- added SW1: SW_Push, symbol Switch:SW_Push
- added U2: W25Q16JVSS, Package_SO:SOIC-8_5.3x5.3mm_P1.27mm, symbol Memory_Flash:W25Q16JVSS
- added U3: RP2040, Package_DFN_QFN:QFN-56-1EP_7x7mm_P0.4mm_EP3.2x3.2mm, symbol MCU_RaspberryPi:RP2040
- added U4: NCP1117-3.3_SOT223, Package_TO_SOT_SMD:SOT-223-3_TabPin2, symbol Regulator_Linear:NCP1117-3.3_SOT223
- added X1: X322512MSB4SI, PCM_JLCPCB:CRYSTAL-SMD_4P-L3.2-W2.5-BL, symbol PCM_JLCPCB-Crystals:Crystal, 12MHz, 20pF
Connections:
- net +3V3: now also C10.1, C11.1, C12.1, C3.1, C4.1, C5.1, C6.1, C7.1, C8.1, C9.1, R5.1, U2.8 (VCC), U3.1 (IOVDD), U3.10 (IOVDD), U3.22 (IOVDD), U3.23 (DVDD), U3.33 (IOVDD), U3.42 (IOVDD), U3.44 (VREG_VIN), U3.45 (VREG_VOUT), U3.49 (IOVDD), U3.50 (DVDD), U4.2 (VO)
- net GND: now also C10.2, C11.2, C12.2, C13.2, C14.2, C15.2, C16.1, C17.1, C3.2, C4.2, C5.2, C6.2, C7.2, C8.2, C9.2, SW1.1, U4.1 (GND), X1.2 (GND), X1.4 (GND)
- net USB_D+: now also R4.1, U3.47 (USB_DP); no longer J1.A6 (D+), J1.B6 (D+)
- net USB_D-: now also R3.1, U3.46 (USB_DM); no longer J1.A7 (D-), J1.B7 (D-)
- net VBUS: now also U4.3 (VI)
- new net: J1.A6 (D+), J1.B6 (D+), R4.2
- new net: J1.A7 (D-), J1.B7 (D-), R3.2
- new net: C17.2, R7.1, X1.1 (OSC)
- new net: R6.1, SW1.2
- new net +1V1: C13.1, C14.1, C15.1, U3.43 (ADC_AVDD), U3.48 (USB_VDD)
- new net GPIO_00: U3.2 (GPIO0)
- new net GPIO_01: U3.3 (GPIO1)
- new net GPIO_02: U3.4 (GPIO2)
- new net GPIO_03: U3.5 (GPIO3)
- new net QSPI_SCLK: U2.6 (CLK), U3.52 (QSPI_SCLK)
- new net QSPI_SD0: U2.5 (DI/IO_{0}), U3.53 (QSPI_SD0)
- new net QSPI_SD1: U2.2 (DO/IO_{1}), U3.55 (QSPI_SD1)
- new net QSPI_SD2: U2.3 (~{WP}/IO_{2}), U3.54 (QSPI_SD2)
- new net QSPI_SD3: U2.7 (~{HOLD}/~{RESET}/IO_{3}), U3.51 (QSPI_SD3)
- new net QSPI_SS: R5.2, R6.2, U2.1 (~{CS}), U3.56 (~{QSPI_SS})
- new net XIN: C16.2, U3.20 (XIN), X1.3 (OSC)
- new net XOUT: R7.2, U3.21 (XOUT)
Other:
- note added: "Crystal Oscillator"
- note added: "Flash Storage"
- note added: "Power Decoupling"
- note added: "RP2040"

Commit message: even more pcb work
Parts:
- added SW2, SW3, SW4, SW5: SW_Push, symbol Switch:SW_Push
Connections:
- net GND: now also SW2.1, SW3.1, SW4.1, SW5.1
- net GPIO_00: now also SW2.2
- net GPIO_01: now also SW3.2
- net GPIO_02: now also SW4.2
- net GPIO_03: now also SW5.2
Other:
- note added: "DDR Buttons"

Commit message: more pcb stuff yay
Parts:
- SW_East: renamed from SW2; footprint (none) -> andrews_lib:DDR_PAD_CONTACT
- SW_North: renamed from SW3; footprint (none) -> andrews_lib:DDR_PAD_CONTACT
- SW_South: renamed from SW5; footprint (none) -> andrews_lib:DDR_PAD_CONTACT
- SW_West: renamed from SW4; footprint (none) -> andrews_lib:DDR_PAD_CONTACT
- renumbered U3 to RP2040
Changed lines of the file:
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@@
 		(dnp no)
 		(fields_autoplaced yes)
-		(property "Reference" "U3"
+		(property "Reference" "RP2040"
 			(at 58.0233 182.88 0)
 			(show_name no)
@@
 			(project "pcb"
 				(path "/e7f534c9-288b-42e9-bbd1-9a18eff38983"
-					(reference "U3")
+					(reference "RP2040")
 					(unit 1)
 				)
@@
 		(dnp no)
 		(fields_autoplaced yes)
-		(property "Reference" "SW4"
+		(property "Reference" "SW_West"
 			(at 120.65 123.19 0)
 			(show_name no)
@@
 			)
 		)
-		(property "Footprint" ""
+		(property "Footprint" "andrews_lib:DDR_PAD_CONTACT"
 			(at 120.65 133.35 0)
 			(hide yes)
@@
 			(project "pcb"
 				(path "/e7f534c9-288b-42e9-bbd1-9a18eff38983"
-					(reference "SW4")
+					(reference "SW_West")
 					(unit 1)
 				)
@@
 		(dnp no)
 		(fields_autoplaced yes)
-		(property "Reference" "SW2"
+		(property "Reference" "SW_East"
 			(at 120.65 102.87 0)
 			(show_name no)
@@
 			)
 		)
-		(property "Footprint" ""
+		(property "Footprint" "andrews_lib:DDR_PAD_CONTACT"
 			(at 120.65 113.03 0)
 			(hide yes)
@@
 			(project "pcb"
 				(path "/e7f534c9-288b-42e9-bbd1-9a18eff38983"
-					(reference "SW2")
+					(reference "SW_East")
 					(unit 1)
 				)
@@
 		(dnp no)
 		(fields_autoplaced yes)
-		(property "Reference" "SW3"
+		(property "Reference" "SW_North"
 			(at 120.65 113.03 0)
 			(show_name no)
@@
 			)
 		)
-		(property "Footprint" ""
+		(property "Footprint" "andrews_lib:DDR_PAD_CONTACT"
 			(at 120.65 123.19 0)
 			(hide yes)
@@
 			(project "pcb"
 				(path "/e7f534c9-288b-42e9-bbd1-9a18eff38983"
-					(reference "SW3")
+					(reference "SW_North")
 					(unit 1)
 				)
@@
 		(dnp no)
 		(fields_autoplaced yes)
-		(property "Reference" "SW5"
+		(property "Reference" "SW_South"
 			(at 120.65 133.35 0)
 			(show_name no)
@@
 			)
 		)
-		(property "Footprint" ""
+		(property "Footprint" "andrews_lib:DDR_PAD_CONTACT"
 			(at 120.65 143.51 0)
 			(hide yes)
@@
 			(project "pcb"
 				(path "/e7f534c9-288b-42e9-bbd1-9a18eff38983"
-					(reference "SW5")
+					(reference "SW_South")
 					(unit 1)
 				)

Commit message: started routing pcb
Parts:
- renumbered U2 to Flash_Storage, SW_East to SW_East1, SW_North to SW_North1, SW_South to SW_South1, SW_West to SW_West1
Changed lines of the file:
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@@
 		(dnp no)
 		(fields_autoplaced yes)
-		(property "Reference" "SW_West"
+		(property "Reference" "SW_West1"
 			(at 120.65 123.19 0)
 			(show_name no)
@@
 			(project "pcb"
 				(path "/e7f534c9-288b-42e9-bbd1-9a18eff38983"
-					(reference "SW_West")
+					(reference "SW_West1")
 					(unit 1)
 				)
@@
 		(dnp no)
 		(fields_autoplaced yes)
-		(property "Reference" "SW_East"
+		(property "Reference" "SW_East1"
 			(at 120.65 102.87 0)
 			(show_name no)
@@
 			(project "pcb"
 				(path "/e7f534c9-288b-42e9-bbd1-9a18eff38983"
-					(reference "SW_East")
+					(reference "SW_East1")
 					(unit 1)
 				)
@@
 		(dnp no)
 		(fields_autoplaced yes)
-		(property "Reference" "SW_North"
+		(property "Reference" "SW_North1"
 			(at 120.65 113.03 0)
 			(show_name no)
@@
 			(project "pcb"
 				(path "/e7f534c9-288b-42e9-bbd1-9a18eff38983"
-					(reference "SW_North")
+					(reference "SW_North1")
 					(unit 1)
 				)
@@
 		(dnp no)
 		(fields_autoplaced yes)
-		(property "Reference" "SW_South"
+		(property "Reference" "SW_South1"
 			(at 120.65 133.35 0)
 			(show_name no)
@@
 			(project "pcb"
 				(path "/e7f534c9-288b-42e9-bbd1-9a18eff38983"
-					(reference "SW_South")
+					(reference "SW_South1")
 					(unit 1)
 				)
@@
 		(dnp no)
 		(fields_autoplaced yes)
-		(property "Reference" "U2"
+		(property "Reference" "Flash_Storage"
 			(at 250.19 43.1799 0)
 			(show_name no)
@@
 			(project "pcb"
 				(path "/e7f534c9-288b-42e9-bbd1-9a18eff38983"
-					(reference "U2")
-					(unit 1)
-				)
+					(reference "Flash_Storage")
+					(unit 1)
+				)

Commit message: saving things for the night
Parts:
- added SW_Menu, SW_Start: SW_Push, symbol Switch:SW_Push
- renumbered Flash_Storage to Flash_Storage1
Connections:
- net GND: now also SW_Menu.1, SW_Start.1
- net GPIO_04: now reaches RP2040.6 (GPIO4)
- net GPIO_04: now also SW_Start.2
- net GPIO_05: now reaches RP2040.7 (GPIO5)
- net GPIO_05: now also SW_Menu.2
Other:
- note added: "ANDREW IS COOL"
- note added: "Extra Buttons"

Commit message: working on pcb even more
Parts:
- SW_East1, SW_South1: footprint andrews_lib:DDR_PAD_CONTACT -> andrews_lib:DDR_BUTTON_2_M
- SW_North1, SW_West1: footprint andrews_lib:DDR_PAD_CONTACT -> andrews_lib:DDR_BUTTON_2
- renumbered SW_Menu to SW_Menu1, SW_Start to SW_Start1
Connections:
- net GND: now also Flash_Storage1.4 (GND), RP2040.57 (GND)
- no-connect marks 0 -> 30
Other:
- company: (none) -> Andrew Cromar
- title: (none) -> Stepminia

Commit message: working on pcb even more
Parts:
- SW1, SW_Menu1, SW_Start1: footprint (none) -> andrews_lib:Tactile_Switch_4.2x3.2
Connections:
- net GPIO_01: now also SW_Start1.2; no longer SW_North1.2
- net GPIO_02: now also SW_Menu1.2; no longer SW_West1.2
- net GPIO_03: now also SW_North1.2; no longer SW_South1.2
- net GPIO_04: now also SW_West1.2; no longer SW_Start1.2
- net GPIO_05: now also SW_South1.2; no longer SW_Menu1.2
Changed lines of the file:
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@@
 	(rectangle
 		(start 190.5 15.24)
-		(end 264.16 59.69)
+		(end 264.16 66.04)
 		(stroke
 			(width 0)
@@
 		)
 	)
+	(global_label "GPIO_05"
+		(shape bidirectional)
+		(at 115.57 138.43 180)
+		(fields_autoplaced yes)
+		(effects
+			(font
+				(size 1.27 1.27)
+			)
+			(justify right)
+		)
+		(property "Intersheetrefs" "${INTERSHEET_REFS}"
+			(at 103.6116 138.43 0)
+			(hide yes)
+			(show_name no)
+			(do_not_autoplace no)
+			(effects
+				(font
+					(size 1.27 1.27)
+				)
+				(justify right)
+			)
+		)
+	)
 	(global_label "XOUT"
 		(shape input)
@@
 		)
 	)
-	(global_label "GPIO_01"
-		(shape bidirectional)
-		(at 115.57 118.11 180)
-		(fields_autoplaced yes)
-		(effects
-			(font
-				(size 1.27 1.27)
-			)
-			(justify right)
-		)
-		(property "Intersheetrefs" "${INTERSHEET_REFS}"
-			(at 103.6116 118.11 0)
-			(hide yes)
-			(show_name no)
-			(do_not_autoplace no)
-			(effects
-				(font
-					(size 1.27 1.27)
-				)
-				(justify right)
-			)
-		)
-	)
-	(global_label "GPIO_04"
-		(shape bidirectional)
-		(at 115.57 166.37 180)
-		(fields_autoplaced yes)
-		(effects
-			(font
-				(size 1.27 1.27)
-			)
-			(justify right)
-		)
-		(property "Intersheetrefs" "${INTERSHEET_REFS}"
-			(at 103.6116 166.37 0)
-			(hide yes)
-			(show_name no)
-			(do_not_autoplace no)
-			(effects
-				(font
-					(size 1.27 1.27)
-				)
-				(justify right)
-			)
-		)
-	)
 	(global_label "GPIO_00"
 		(shape bidirectional)
@@
 		)
 	)
-	(global_label "GPIO_03"
+	(global_label "GPIO_01"
 		(shape bidirectional)
-		(at 115.57 138.43 180)
+		(at 115.57 166.37 180)
 		(fields_autoplaced yes)
 		(effects
@@
 		)
 		(property "Intersheetrefs" "${INTERSHEET_REFS}"
-			(at 103.6116 138.43 0)
+			(at 103.6116 166.37 0)
 			(hide yes)
 			(show_name no)
@@
 		)
 	)
-	(global_label "QSPI_SD3"
+	(global_label "GPIO_03"
 		(shape bidirectional)
-		(at 30.48 146.05 180)
+		(at 115.57 118.11 180)
 		(fields_autoplaced yes)
 		(effects
@@
 		)
 		(property "Intersheetrefs" "${INTERSHEET_REFS}"
-			(at 17.3121 146.05 0)
+			(at 103.6116 118.11 0)
 			(hide yes)
 			(show_name no)
@@
 		)
 	)
-	(global_label "QSPI_SCLK"
-		(shape input)
-		(at 228.6 39.37 180)
+	(global_label "QSPI_SD3"
+		(shape bidirectional)
+		(at 30.48 146.05 180)
 		(fields_autoplaced yes)
 		(effects
@@
 		)
 		(property "Intersheetrefs" "${INTERSHEET_REFS}"
-			(at 215.4548 39.37 0)
+			(at 17.3121 146.05 0)
 			(hide yes)
 			(show_name no)
@@
 		)
 	)
-	(global_label "GPIO_05"
-		(shape bidirectional)
-		(at 115.57 176.53 180)
+	(global_label "QSPI_SCLK"
+		(shape input)
+		(at 228.6 39.37 180)
 		(fields_autoplaced yes)
 		(effects
@@
 		)
 		(property "Intersheetrefs" "${INTERSHEET_REFS}"
-			(at 103.6116 176.53 0)
+			(at 215.4548 39.37 0)
 			(hide yes)
 			(show_name no)
@@
 		)
 	)
+	(global_label "GPIO_04"
+		(shape bidirectional)
+		(at 115.57 128.27 180)
+		(fields_autoplaced yes)
+		(effects
+			(font
+				(size 1.27 1.27)
+			)
+			(justify right)
+		)
+		(property "Intersheetrefs" "${INTERSHEET_REFS}"
+			(at 103.6116 128.27 0)
+			(hide yes)
+			(show_name no)
+			(do_not_autoplace no)
+			(effects
+				(font
+					(size 1.27 1.27)
+				)
+				(justify right)
+			)
+		)
+	)
 	(global_label "XOUT"
 		(shape output)
@@
 		)
 	)
-	(global_label "GPIO_02"
+	(global_label "USB_D+"
 		(shape bidirectional)
-		(at 115.57 128.27 180)
+		(at 30.48 125.73 180)
 		(fields_autoplaced yes)
 		(effects
@@
 		)
 		(property "Intersheetrefs" "${INTERSHEET_REFS}"
-			(at 103.6116 128.27 0)
+			(at 18.7635 125.73 0)
 			(hide yes)
 			(show_name no)
@@
 		)
 	)
-	(global_label "USB_D+"
+	(global_label "QSPI_SD2"
 		(shape bidirectional)
-		(at 30.48 125.73 180)
+		(at 228.6 46.99 180)
 		(fields_autoplaced yes)
 		(effects
@@
 		)
 		(property "Intersheetrefs" "${INTERSHEET_REFS}"
-			(at 18.7635 125.73 0)
+			(at 215.4321 46.99 0)
 			(hide yes)
 			(show_name no)
@@
 		)
 	)
-	(global_label "QSPI_SD2"
+	(global_label "GPIO_02"
 		(shape bidirectional)
-		(at 228.6 46.99 180)
+		(at 115.57 176.53 180)
 		(fields_autoplaced yes)
 		(effects
@@
 		)
 		(property "Intersheetrefs" "${INTERSHEET_REFS}"
-			(at 215.4321 46.99 0)
+			(at 103.6116 176.53 0)
 			(hide yes)
 			(show_name no)
@@
 			)
 		)
-		(property "Footprint" ""
+		(property "Footprint" "andrews_lib:Tactile_Switch_4.2x3.2"
 			(at 120.65 181.61 0)
 			(hide yes)
@@
 			)
 		)
-		(property "Footprint" ""
+		(property "Footprint" "andrews_lib:Tactile_Switch_4.2x3.2"
 			(at 120.65 171.45 0)
 			(hide yes)
@@
 			)
 		)
-		(property "Footprint" ""
+		(property "Footprint" "andrews_lib:Tactile_Switch_4.2x3.2"
 			(at 200.66 31.75 0)
 			(hide yes)

Commit message: work on it yay
Parts:
- SW1, SW_Menu1, SW_Start1: footprint andrews_lib:Tactile_Switch_4.2x3.2 -> Andrews_Library:Tactile_Switch_4.2x3.2
Changed lines of the file:
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@@
 			)
 		)
-		(property "Footprint" "andrews_lib:Tactile_Switch_4.2x3.2"
+		(property "Footprint" "Andrews_Library:Tactile_Switch_4.2x3.2"
 			(at 120.65 181.61 0)
 			(hide yes)
@@
 			)
 		)
-		(property "Footprint" "andrews_lib:Tactile_Switch_4.2x3.2"
+		(property "Footprint" "Andrews_Library:Tactile_Switch_4.2x3.2"
 			(at 120.65 171.45 0)
 			(hide yes)
@@
 			)
 		)
-		(property "Footprint" "andrews_lib:Tactile_Switch_4.2x3.2"
+		(property "Footprint" "Andrews_Library:Tactile_Switch_4.2x3.2"
 			(at 200.66 31.75 0)
 			(hide yes)
