File: pcb/pcb.kicad_sch (KiCad schematic)
At the start: 20 parts, among them U1 1117-3.3

Commit message: working on ddr contacts n stuff
Parts:
- added U2: NORTH, Andrews_Library:DDR_CONTACT, symbol Andrews_Library:DDR_CONTACT
- added U3: SOUTH, Andrews_Library:DDR_CONTACT, symbol Andrews_Library:DDR_CONTACT
- added U4: EAST, Andrews_Library:DDR_CONTACT, symbol Andrews_Library:DDR_CONTACT
- added U5: WEST, Andrews_Library:DDR_CONTACT, symbol Andrews_Library:DDR_CONTACT
Connections:
- net GND: now also U2.1 (GND), U3.1 (GND), U4.1 (GND), U5.1 (GND)

Commit message: work on schematic more
Parts:
- added U6: RP2040, Package_DFN_QFN:QFN-56-1EP_7x7mm_P0.4mm_EP3.2x3.2mm, symbol MCU_RaspberryPi:RP2040
Connections:
- net +1V1: now also U6.43 (ADC_AVDD), U6.48 (USB_VDD)
- net +3V3: now also U6.1 (IOVDD), U6.10 (IOVDD), U6.22 (IOVDD), U6.23 (DVDD), U6.33 (IOVDD), U6.42 (IOVDD), U6.44 (VREG_VIN), U6.45 (VREG_VOUT), U6.49 (IOVDD), U6.50 (DVDD)
- net GND: now also U6.57 (GND)
- net USB_DN: now also U6.46 (USB_DM)
- net USB_DP: now also U6.47 (USB_DP)
- net GPIO-17: now reaches U3.2 (GPIO)
- net GPIO-17: now also U6.28 (GPIO17)
- net GPIO-18: now reaches U4.2 (GPIO)
- net GPIO-18: now also U6.29 (GPIO18)

Commit message: working on schematic now
Parts:
- added C15: 0.1uF, Capacitor_SMD:C_0201_0603Metric, symbol Device:C
- added R5: 10k, Resistor_SMD:R_0201_0603Metric, symbol Device:R
- added R6: 1k, Resistor_SMD:R_0201_0603Metric, symbol Device:R
- added U7: (no value), symbol Andrews_Library:LCSC_W25Q16JVSSIQ_C131025
Connections:
- net +3V3: now also C15.1, R5.1, U7.8 (VCC)
- net GND: now also C15.2
- net QSPI_SD3: now reaches U6.51 (QSPI_SD3)
- net QSPI_SD3: now also U7.7 (HOLD/RESET/IO₃)
- net QSPI_SCLK: now reaches U6.52 (QSPI_SCLK)
- net QSPI_SCLK: now also U7.6 (CLK)
- net QSPI_SD0: now reaches U6.53 (QSPI_SD0)
- net QSPI_SD0: now also U7.5 (DI/IO₀)
- net QSPI_SD2: now reaches U6.54 (QSPI_SD2)
- net QSPI_SD2: now also U7.3 (WP/IO₂)
- net QSPI_SD1: now reaches U6.55 (QSPI_SD1)
- net QSPI_SD1: now also U7.2 (DO/IO₁)
- net QSPI_SS: now reaches U6.56 (~{QSPI_SS})
- net QSPI_SS: now also R5.2, R6.1, U7.1 (/CS)

Commit message: work on schematic
Parts:
- added U8: (no value), Andrews_Library:LCSC_TS-1089S-02526_C455282, symbol Andrews_Library:LCSC_TS-1089S-02526_C455282
- U7: footprint (none) -> Andrews_Library:LCSC_W25Q16JVSSIQ_C131025
Connections:
- net GND: now also U8.3 (OUT1), U8.4 (OUT2)
- net at R6.2: now also U8.1 (IN1), U8.2 (IN2)
Other:
- note added: "Contacts"
- note added: "Flash Storage"
- moved on the sheet: C15, R5, R6, U2, U3, U4, U5, U7

Commit message: even more pcb stuff
Parts:
- U2, U4: footprint Andrews_Library:DDR_CONTACT -> Andrews_Library:DDR_CONTACT_MIRROR
Connections:
- net GND: now also U7.4 (GND)
- net GPIO-25: now reaches U2.2 (GPIO)
- net GPIO-25: now also U6.37 (GPIO25)
- net GPIO-12: now reaches U5.2 (GPIO)
- net GPIO-12: now also U6.15 (GPIO12)
Changed lines of the file:
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@@
 	(wire
 		(pts
+			(xy 171.45 85.09) (xy 171.45 86.36)
+		)
+		(stroke
+			(width 0)
+			(type default)
+		)
+	)
+	(wire
+		(pts
 			(xy 171.45 36.83) (xy 177.8 36.83)
 		)
@@
 	(wire
 		(pts
+			(xy 171.45 86.36) (xy 170.18 86.36)
+		)
+		(stroke
+			(width 0)
+			(type default)
+		)
+	)
+	(wire
+		(pts
 			(xy 35.56 48.26) (xy 35.56 50.8)
 		)
@@
 		)
 	)
+	(global_label "GPIO-25"
+		(shape input)
+		(at 87.63 163.83 0)
+		(fields_autoplaced yes)
+		(effects
+			(font
+				(size 1.27 1.27)
+			)
+			(justify left)
+		)
+		(property "Intersheetrefs" "${INTERSHEET_REFS}"
+			(at 99.0819 163.83 0)
+			(hide yes)
+			(show_name no)
+			(do_not_autoplace no)
+			(effects
+				(font
+					(size 1.27 1.27)
+				)
+				(justify left)
+			)
+		)
+	)
 	(global_label "GPIO-17"
 		(shape input)
@@
 		)
 	)
+	(global_label "GPIO-12"
+		(shape input)
+		(at 87.63 130.81 0)
+		(fields_autoplaced yes)
+		(effects
+			(font
+				(size 1.27 1.27)
+			)
+			(justify left)
+		)
+		(property "Intersheetrefs" "${INTERSHEET_REFS}"
+			(at 99.0819 130.81 0)
+			(hide yes)
+			(show_name no)
+			(do_not_autoplace no)
+			(effects
+				(font
+					(size 1.27 1.27)
+				)
+				(justify left)
+			)
+		)
+	)
 	(global_label "GPIO-17"
 		(shape input)
@@
 		)
 	)
+	(global_label "GPIO-25"
+		(shape input)
+		(at 222.25 29.21 180)
+		(fields_autoplaced yes)
+		(effects
+			(font
+				(size 1.27 1.27)
+			)
+			(justify right)
+		)
+		(property "Intersheetrefs" "${INTERSHEET_REFS}"
+			(at 210.7981 29.21 0)
+			(hide yes)
+			(show_name no)
+			(do_not_autoplace no)
+			(effects
+				(font
+					(size 1.27 1.27)
+				)
+				(justify right)
+			)
+		)
+	)
 	(global_label "USB_DN"
 		(shape bidirectional)
@@
 		)
 	)
+	(global_label "GPIO-12"
+		(shape input)
+		(at 222.25 55.88 180)
+		(fields_autoplaced yes)
+		(effects
+			(font
+				(size 1.27 1.27)
+			)
+			(justify right)
+		)
+		(property "Intersheetrefs" "${INTERSHEET_REFS}"
+			(at 210.7981 55.88 0)
+			(hide yes)
+			(show_name no)
+			(do_not_autoplace no)
+			(effects
+				(font
+					(size 1.27 1.27)
+				)
+				(justify right)
+			)
+		)
+	)
 	(symbol
 		(lib_id "power:+3V3")
@@
 			)
 		)
-		(property "Footprint" "Andrews_Library:DDR_CONTACT"
+		(property "Footprint" "Andrews_Library:DDR_CONTACT_MIRROR"
 			(at 229.87 27.94 0)
 			(hide yes)
@@
 			)
 		)
-		(property "Footprint" "Andrews_Library:DDR_CONTACT"
+		(property "Footprint" "Andrews_Library:DDR_CONTACT_MIRROR"
 			(at 229.87 45.72 0)
 			(hide yes)
@@
 					(unit 1)
 				)
+			)
+		)
+	)
+	(symbol
+		(lib_id "power:GND")
+		(at 170.18 86.36 0)
+		(unit 1)
+		(body_style 1)
+		(exclude_from_sim no)
+		(in_bom yes)
+		(on_board yes)
+		(in_pos_files yes)
+		(dnp no)
+		(fields_autoplaced yes)
+		(property "Reference" "#PWR020"
+			(at 170.18 92.71 0)
+			(hide yes)
+			(show_name no)
+			(do_not_autoplace no)
+			(effects
+				(font
+					(size 1.27 1.27)
+				)
+			)
+		)
+		(property "Value" "GND"
+			(at 170.18 91.44 0)
+			(show_name no)
+			(do_not_autoplace no)
+			(effects
+				(font
+					(size 1.27 1.27)
+				)
+			)
+		)
+		(property "Footprint" ""
+			(at 170.18 86.36 0)
+			(hide yes)
+			(show_name no)
+			(do_not_autoplace no)
+			(effects
+				(font
+					(size 1.27 1.27)
+				)
+			)
+		)
+		(property "Datasheet" ""
+			(at 170.18 86.36 0)
+			(hide yes)
+			(show_name no)
+			(do_not_autoplace no)
+			(effects
+				(font
+					(size 1.27 1.27)
+				)
+			)
+		)
+		(property "Description" "Power symbol creates a global label with name \"GND\" , ground"
+			(at 170.18 86.36 0)
+			(hide yes)
+			(show_name no)
+			(do_not_autoplace no)
+			(effects
+				(font
+					(size 1.27 1.27)
+				)
+			)
+		)
+		(pin "1"
+		)
+		(instances
+			(project "pcb"
+				(path "/37969d75-6775-4969-b3c5-2af34bbf809f"
+					(reference "#PWR020")
+					(unit 1)
+				)
