File: pcb/RP2040_minimal_r2/RP2040_minimal_r2.kicad_pcb (KiCad board)
At the start: 2 copper layers, 75 x 75 mm, 34 parts, among them J2 Conn_01x02, J3 USB_C_Receptacle, SW1 DDR_North, SW2 DDR_South, SW3 DDR_East, SW4 DDR_West, U1 NCP1117-3.3_SOT223, U2 W25Q128JVS, U3 RP2040, Y1 ABM8-272-T3

Commit message: add rest of lcsc numbers
Parts:
- R2: value DNF -> 10k
