File: pcb/simple/pcb/pcb.kicad_sch (KiCad schematic)
At the start: 0 parts

Commit message: finish pcb
Parts:
- added SW1: DDR_North, Andrews_Library:DDR_CONTACT, symbol Switch:SW_Push
- added SW2: DDR_East, Andrews_Library:DDR_CONTACT, symbol Switch:SW_Push
- added SW3: DDR_South, Andrews_Library:DDR_CONTACT_MIRROR, symbol Switch:SW_Push
- added SW4: DDR_West, Andrews_Library:DDR_CONTACT_MIRROR, symbol Switch:SW_Push
- added SW5: SW_Pause, Button_Switch_THT:SW_PUSH_6mm, symbol Switch:SW_Push
- added SW6: SW_Start, Button_Switch_THT:SW_PUSH_6mm, symbol Switch:SW_Push
- added U1: RP2040-ZERO, RP2040-ZERO:MODULE_RP2040-ZERO, symbol RP2040-ZERO:RP2040-ZERO
Connections:
- new net GND: SW1.2, SW2.2, SW3.2, SW4.2, SW5.2, SW6.2, U1.22 (GND)
- new net GPIO3: SW5.1, U1.4 (GP3)
- new net GPIO4: SW6.1, U1.5 (GP4)
- new net GPIO5: SW1.1, U1.6 (GP5)
- new net GPIO6: SW2.1, U1.7 (GP6)
- new net GPIO7: SW3.1, U1.8 (GP7)
- new net GPIO8: SW4.1, U1.9 (GP8)
- no-connect marks 0 -> 16
Other:
- note added: "Buttons"
- note added: "MCU"
- company: (none) -> Andrew Cromar
- title: (none) -> Stepmini PCB
